File: kicad-wifi/vfo-pcb.kicad_pcb (KiCad board)
At the start: 2 copper layers, 108.4 x 79.9 mm, 97 parts, among them J1 Rotery Encoder1, J10 Link-out 1-2, J11 Link-out 1-0, J12 Link-out 2-0, J13 Link-out 2-2, J14 Link-out 2-1, J15 Link-out 1-1, J2 Rotery Encoder2, J3 Analog in 3-6, J4 RxTx, J5 V12, J6 ESP32L, J7 ESP32R, J8 ILI9341, J9 Conn_01x07_Female, Q1 BFR92, Q2 BFR92, Q3 BFR92, Q4 BFR92, Q5 BFR92, Q6 BFR92, SW1 Rotary_Encoder_Switch, U1 AMS1117, U2 LM2576HVS-ADJ, U3 Si5351A-B-GT, U4 Si5351A-B-GT, Y1 Crystal, Y2 Crystal

Commit message: update wifi pcb
Parts:
- added C20: 100n, Capacitor_SMD:C_1206_3216Metric_Pad1.42x1.75mm_HandSolder, F.Cu at (129.3, 124.0)
- added C21: 100n, Capacitor_SMD:C_1206_3216Metric_Pad1.42x1.75mm_HandSolder, F.Cu at (105.4, 124.0)
- added C22: 100n, Capacitor_SMD:C_1206_3216Metric_Pad1.42x1.75mm_HandSolder, F.Cu at (90.2, 129.3)
- added C23: 100n, Capacitor_SMD:C_1206_3216Metric_Pad1.42x1.75mm_HandSolder, F.Cu at (88.6, 125.2)
- added C24: 100n, Capacitor_SMD:C_1206_3216Metric_Pad1.42x1.75mm_HandSolder, F.Cu at (74.9, 126.2)
- added C25: 100n, Capacitor_SMD:C_1206_3216Metric_Pad1.42x1.75mm_HandSolder, F.Cu at (51.1, 125.2)
- R26, R27, R31: value 33 -> 200
- R33, R34, R37: value 150 -> 68
- moved C8 22.6 mm to (131.6, 84.1), turned to 180 degrees
- moved R34 20.0 mm to (45.0, 120.1), turned to 90 degrees
- moved R36 11.1 mm to (91.4, 125.2), turned to 270 degrees
- moved R38 5.41 mm to (105.4, 118.6)
- moved C10 3.31 mm to (142.4, 88.3)
- moved C6 3.31 mm to (130.1, 88.3)
- moved L1 1.78 mm to (140.5, 106.2)
- moved C12 1.52 mm to (130.8, 95.5)
- moved R39 1.52 mm to (137.2, 95.5)
- moved R40 1.52 mm to (142.9, 95.5)
- moved R37 1.51 mm to (77.5, 126.2)
- moved J13 0.50 mm to (56.6, 125.7)
Connections:
- J10 pad 1: Net-(J10-Pad1) -> Net-(C22-Pad2)
- J11 pad 1: Net-(J11-Pad1) -> Net-(C20-Pad2)
- J12 pad 1: Net-(J12-Pad1) -> Net-(C23-Pad2)
- J13 pad 1: Net-(J13-Pad1) -> Net-(C25-Pad2)
- J14 pad 1: Net-(J14-Pad1) -> Net-(C24-Pad2)
- J15 pad 1: Net-(J15-Pad1) -> Net-(C21-Pad2)
- R26 pad 2: Net-(J12-Pad1) -> Net-(C23-Pad1)
- R27 pad 2: Net-(J13-Pad1) -> Net-(C25-Pad1)
- R28 pad 2: Net-(J11-Pad1) -> Net-(C20-Pad1)
- R30 pad 2: Net-(J10-Pad1) -> Net-(C22-Pad1)
- R31 pad 2: Net-(J14-Pad1) -> Net-(C24-Pad1)
- R32 pad 1: Net-(J11-Pad1) -> Net-(C20-Pad1)
- R33 pad 1: Net-(J12-Pad1) -> Net-(C23-Pad1)
- R34 pad 1: Net-(J13-Pad1) -> Net-(C25-Pad1)
- R35 pad 2: Net-(J15-Pad1) -> Net-(C21-Pad1)
- R36 pad 1: Net-(J10-Pad1) -> Net-(C22-Pad1)
- R37 pad 1: Net-(J14-Pad1) -> Net-(C24-Pad1)
- R38 pad 1: Net-(J15-Pad1) -> Net-(C21-Pad1)
- SW1 pad MP: GND -> (no net)
Routing:
- net Net-(J12-Pad1): track 18.2 -> 0.00 mm
- net Net-(J13-Pad1): track 16.6 -> 0.00 mm
- net Net-(J14-Pad1): track 15.2 -> 0.00 mm
- net Net-(J10-Pad1): track 14.4 -> 0.00 mm
- net Net-(C23-Pad1): track 0.00 -> 13.8 mm
- net Net-(J15-Pad1): track 11.3 -> 0.00 mm
- net Net-(C25-Pad1): track 0.00 -> 9.40 mm
- net Net-(C22-Pad1): track 0.00 -> 9.39 mm
- net Net-(C21-Pad1): track 0.00 -> 9.08 mm
- net Net-(J11-Pad1): track 8.97 -> 0.00 mm
- net Net-(C22-Pad2): track 0.00 -> 8.88 mm
- net Net-(C24-Pad1): track 0.00 -> 8.40 mm
- net Vcc: track 246.0 -> 239.2 mm
- net Net-(C24-Pad2): track 0.00 -> 6.18 mm
- net Net-(C23-Pad2): track 0.00 -> 6.05 mm
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