File: Kicad/vfo-pcb.kicad_pcb (KiCad board)
At the start: 2 copper layers, 108.4 x 79.9 mm, 94 parts, among them J1 Rotery Encoder1, J10 Link-out 1-2, J11 Link-out 1-0, J12 Link-out 2-0, J13 Link-out 2-2, J14 Link-out 2-1, J15 Link-out 1-1, J2 Rotery Encoder2, J3 Analog in 3-6, J4 RxTx, J5 V12, J6 ESP32L, J7 ESP32R, J8 ILI9341, J9 Conn_01x07_Female, Q1 BFR92, Q2 BFR92, Q3 BFR92, Q4 BFR92, Q5 BFR92, Q6 BFR92, SW1 Rotary_Encoder_Switch, U1 AMS1117, U2 L7805, U3 Si5351A-B-GT, U4 Si5351A-B-GT, Y1 Crystal, Y2 Crystal

Commit message: change debounce
Parts:
- C11, C13, C9: value 10n -> 100n
Connections:
- SW1 pad MP: GND -> (no net)
