File: Kicad-new/ESP32Vfo.kicad_pcb (KiCad board)
At the start: 4 copper layers, 100 x 57 mm, 124 parts, among them J1 ILI9341, J10 USB_C_Receptacle_USB2.0, J11 Link-out 1-0, J12 Link-out 1-0, J13 Link-out 1-1, J14 Link-out 1-1, J2 5V, J3 Jtag, J4 I2C, J5 Relais, J6 I2C, J7 Encoders, J8 Encoders, J9 Analog in 3-6, Q1 2N3904_SOT23, Q2 2N3904_SOT23, Q3 BFR92, Q4 BFR92, Q5 BFR92, Q6 BFR92, Q7 2N3904_SOT23, Q8 2N3904_SOT23, SW1 SW_Push, SW2 SW_Push, U1 LM1117-3.3, U2 ESP32-WROOM-32D, U3 PCF8574A, U4 CP2102N-A01-GQFN28, U5 TCA9548APWR, U6 Si5351A-B-GT, U7 Si5351A-B-GT, Y1 Crystal, Y2 Crystal

Commit message: new pcb
Parts:
- added R47: 2.2k, Resistor_SMD:R_0805_2012Metric, F.Cu at (96.5, 61.1)
- added R48: 2.2k, Resistor_SMD:R_0805_2012Metric, F.Cu at (94.1, 61.1)
Connections:
- J10 pad S1: (no net) -> Net-(J10-PadS1)
- U5 pad 17: Net-(U5-Pad17) -> SDA_2
- U5 pad 18: Net-(U5-Pad18) -> SCL_2
- U6 pad 4: SCL_1 -> SCL_2
- U6 pad 5: SDA_1 -> SDA_2
- Y1 pad 4: GND -> (no net)
- Y2 pad 4: GND -> (no net)
Routing:
- net SCL_2: track 0.00 -> 38.4 mm
- net SDA_2: track 0.00 -> 35.8 mm
- net SDA_1: track 51.1 -> 33.8 mm
- net SCL_1: track 48.4 -> 38.8 mm
- net GND: track 19.3 -> 19.6 mm, vias 63 -> 61
- net V33: vias 48 -> 50
- net (no net): vias 0 -> 2

Commit message: update pcb
Parts:
- removed the R31 at (97.4, 76.2)
- SW1: footprint ESP32_TouchDown_lib:TS-1088R-02526 -> ESP32VFO:TS-1088R-02526
Connections:
- J1 pad 11: T_CS -> IO0
- J1 pad 4: V33 -> Reset
- J10 pad S1: Net-(J10-PadS1) -> (no net)
- U2 pad 26: INT -> Reset
- U3 pad 13: INT -> Net-(U3-Pad13)
- U3 pad 16: Net-(U3-Pad16) -> V33
Routing:
- net Reset: track 0.00 -> 46.9 mm, vias 0 -> 3
- net IO0: track 9.98 -> 43.1 mm, vias 0 -> 5
- net INT: track 20.1 -> 0.00 mm, vias 2 -> 0
- net T2: track 14.4 -> 12.2 mm
- net Net-(Q2-Pad1): track 7.84 -> 5.90 mm
- net V33: vias 50 -> 51

Commit message: update pcb
Parts:
- removed C21: 100n, Capacitor_SMD:C_0805_2012Metric
- added D3: PGB1010603MR, digikey-footprints:0603, F.Cu at (54.6, 48.5)
- added D4: PGB1010603MR, digikey-footprints:0603, F.Cu at (57.3, 48.5)
- added R49: 2k2, Resistor_SMD:R_0805_2012Metric, F.Cu at (91.8, 61.1)
- moved C27 4.07 mm to (79.2, 71.0), turned to 180 degrees
- moved R38 2.54 mm to (127.8, 55.8), turned to 180 degrees
- moved R36 2.29 mm to (127.8, 53.3), turned to 0 degrees
Connections:
- J10 pad S1: (no net) -> Net-(J10-PadS1)
- U2 pad 7: A5P -> INT
- U3 pad 13: Net-(U3-Pad13) -> INT
Routing:
- net INT: track 0.00 -> 77.9 mm, vias 0 -> 2
- net A5P: track 23.6 -> 0.00 mm, vias 1 -> 0
- net Net-(Q4-Pad2): track 7.34 -> 2.26 mm
- net V33: track 32.3 -> 35.3 mm
- net D-: track 15.1 -> 16.4 mm
- net GND: track 19.6 -> 20.9 mm, vias 61 -> 64
- net D+: track 14.1 -> 15.1 mm
- net Net-(C31-Pad1): track 4.71 -> 5.54 mm
